File: pcb/mainboard/elflet.brd (EAGLE design)
At the start: 32 x 58 mm, 37 parts, among them J1 ZX62-B-5PA(33), J2 2212S-10SG-36, Q1 IRLML6344TRPBF, Q2 ALS-PT19-315C_L177_TR8, SW1 SKRPACE010, U1 ESP-WROOM-32, U2 ADP3338AKCZ-3.3, U3 OSRB38C9AATILT, U4 BME280

Commit message: initial wiring
Parts:
- J3: value (none) -> STD-PINHD-1X6
- LED3: device OSTBABS4C2B:LRTB-GVTG_99 -> OSTBABS4C2B:OSTBABS4C2B
- Q2: value ALS-PT19-315C_L177_TR8 -> ALS-PT19-315C/L177/TR8
- R1, R10, R14, R2, R3: value 10K(5%) -> 10K(0.1%)
- R11, R12: value 33(5%) -> 33(0.1%)
- R13: value 220(5%) -> 220(0.1%)
- R15: value BCN164A101J7 -> BCN164AB101J7
- R4, R5: value 4.7K(5%) -> 4.7K(0.1%)
- R7: device rcl:R6332 -> gen-discrete:R2512
- R8: value 22K(5%) -> 22K(0.1%)
- R9: value 47(5%) -> 47(0.1%)
- U3: value OSRB38C9AATILT -> OSRB38C9AA
- moved C8 5.24 mm to (6.60, 50.3), turned to 90 degrees
- moved R11 5.08 mm to (29.2, 2.54), turned to 270 degrees
- moved R4 5.06 mm to (4.57, 46.6)
- moved R5 5.06 mm to (6.60, 46.6)
- moved R13 4.60 mm to (24.6, 2.54), turned to 270 degrees
- moved LED3 3.87 mm to (26.0, 8.89)
- moved R1 3.81 mm to (6.35, 15.2), turned to 270 degrees
- moved R12 3.61 mm to (26.9, 2.54), turned to 270 degrees
- moved LED1 2.54 mm to (7.87, 55.5)
- moved C9 1.63 mm to (4.57, 50.3), turned to 90 degrees
- moved R14 1.27 mm to (6.35, 8.89)
- moved U4 1.27 mm to (2.79, 55.9), turned to 270 degrees
- moved C7 0.89 mm to (15.5, 53.8)
Connections:
- net GND: now also U1.GND_B, U1.GND_V
Routing:
- net GND: track 0.00 -> 207.9 mm, vias 0 -> 201
- net +3V3: track 0.00 -> 142.8 mm, vias 0 -> 4
- net BOOT: track 0.00 -> 122.9 mm, vias 0 -> 2
- net +5V: track 0.00 -> 85.8 mm, vias 0 -> 9
- net N$1: track 0.00 -> 79.2 mm
- net AUX_MISO: track 0.00 -> 65.2 mm, vias 0 -> 1
- net AUX_SS: track 0.00 -> 54.0 mm, vias 0 -> 1
- net TXD: track 0.00 -> 46.7 mm, vias 0 -> 1
- net RXD: track 0.00 -> 44.6 mm, vias 0 -> 2
- net SCL: track 0.00 -> 43.1 mm, vias 0 -> 2
- net IRRX: track 0.00 -> 42.5 mm, vias 0 -> 1
- net AUX_SCK: track 0.00 -> 37.5 mm, vias 0 -> 4
- net AUX_MOSI: track 0.00 -> 35.6 mm, vias 0 -> 2
- net SDA: track 0.00 -> 35.2 mm, vias 0 -> 4
- net RESET: track 0.00 -> 34.2 mm, vias 0 -> 3
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- added copper zone on layer 1, net +5V
- added copper zone on layer 16, net +5V
- added copper zone on layer 1, net GND
- added copper zone on layer 16, net GND
